Commit message: Actuators addition

File: #CODES/RobotDog/Robot Final.SLDASM.urdf (robot description, URDF)
Before this commit: robot Robot Final.SLDASM, 9 links, 8 joints
Links:
- link base_link: mass 0.31232 -> 0.312315740063627
- link left_back_leg: mass 0.0130112653193228 -> 0.0130112653193227
- link right_shoulder: mass 0.015764489154619 -> 0.015764
Joints:
- joint left_shoulder_link: origin xyz=0.049406 -0.099056 -0.083518 rpy=-3.1416 0 2.7021 -> xyz=0.0494064879704632 -0.099056323906075 -0.0835183568674249 rpy=-3.14159265358979 0 2.7020575896327

Commit message: Kinematics

File: #CODES/RobotDog/Robot Final.SLDASM.urdf (robot description, URDF)
Before this commit: robot Robot Final.SLDASM, 9 links, 8 joints
Links:
- link base_link: mass 0.312315740063627 -> 0.33418
- link left_back_leg: mass 0.0130112653193227 -> 0.013922
- link left_front_leg: mass 0.0130112653193228 -> 0.013922
- link left_hip: mass 0.001 -> 0.016868
- link left_shoulder: mass 0.015764489154619 -> 0.016868
- link right_back_leg: mass 0.0130112653193228 -> 0.013922
- link right_front_leg: mass 0.0130112653193228 -> 0.013922
- link right_hip: mass 0.0157644891546191 -> 0.016868
- link right_shoulder: mass 0.015764 -> 0.016868
Joints:
- joint left_front_leg_link: origin xyz=0 0.020003 0.0065 rpy=0 0 -1.421 -> xyz=0 0.0200030365383422 0.00649999999999558 rpy=0 0 -1.42102242994654
- joint left_hip_link: axis 0 0 1 -> 0.0 0 1; origin xyz=-0.080372 -0.070493 -0.083518 rpy=-3.1416 0 -2.2041 -> xyz=-0.0803722222962356 -0.0704931866509989 -0.0835183568674255 rpy=-3.14159265358979 0 -2.20414374810614
- joint right_back_leg_link: axis 0 0 1 -> 0.0 0 1; origin xyz=0 0.020003 0.0065 rpy=0 0 -1.0068 -> xyz=0 0.0200030365383461 0.00649999999999981 rpy=0 0 -1.00676371861286
- joint right_front_leg_link: origin xyz=0 0.020003 0.0065 rpy=0 0 0.62485 -> xyz=0 0.020003036538349 0.00650000000000464 rpy=0 0 0.624846439392489
- joint right_hip_link: origin xyz=-0.082726 -0.073575 0.069482 rpy=0 0 0.89496 -> xyz=-0.0827258320400727 -0.0735749478654602 0.0694816431325751 rpy=0 0 0.894961894405035
